File: MixedSignal/3bflashadc.kicad_sch (KiCad schematic)
At the start: 32 parts, among them U11 ADCMP602BRMZ, U12 ADCMP602BRMZ, U13 ADCMP602BRMZ, U14 ADCMP602BRMZ, U15 ADCMP602BRMZ, U16 ADCMP602BRMZ, U17 ADCMP602BRMZ, U18 CDCLVC1108PW, U19 DS90LV012ATMFX

Commit message: passing DRC
Parts:
- removed R33: 100(0.1%), Resistor_SMD:R_0603_1608Metric, symbol Device:R_US
- removed U19: DS90LV012ATMFX, ClockDistributer:PW0016A_N, symbol LVDSReciever:DS90LV012ATMFX
- added C43, C44, C45, C46, C47, C48, C49, C50, C51, C52: 0.1µF Ceramic, Capacitor_SMD:C_0603_1608Metric, symbol Device:C
- U10: renamed from U11; footprint ADCComparator:DGN8_1P89X1P57 -> Package_SO:MSOP-8_3x3mm_P0.65mm
- U11: renamed from U12; footprint ADCComparator:DGN8_1P89X1P57 -> Package_SO:MSOP-8_3x3mm_P0.65mm
- U12: renamed from U13; footprint ADCComparator:DGN8_1P89X1P57 -> Package_SO:MSOP-8_3x3mm_P0.65mm
- U13: renamed from U14; footprint ADCComparator:DGN8_1P89X1P57 -> Package_SO:MSOP-8_3x3mm_P0.65mm
- U14: renamed from U15; footprint ADCComparator:DGN8_1P89X1P57 -> Package_SO:MSOP-8_3x3mm_P0.65mm
- U15: renamed from U16; footprint ADCComparator:DGN8_1P89X1P57 -> Package_SO:MSOP-8_3x3mm_P0.65mm
- U16: renamed from U17; footprint ADCComparator:DGN8_1P89X1P57 -> Package_SO:MSOP-8_3x3mm_P0.65mm
- renumbered C28 to C29, C32 to C31, C34 to C32, C36 to C33, C38 to C34, C40 to C35, C29 to C36, C31 to C37, C33 to C38, C35 to C39, C37 to C40, C39 to C41, C41 to C42, R26 to R29, R28 to R30, R30 to R31, R25 to R33, R27 to R34, R29 to R35, R31 to R36
Connections:
- net +0.3125V: now also C49.1
- net +0.625V: now also C43.1
- net +0.9375V: now also C48.1
- net +1.25V: now also C44.1
- net +1.5625V: now also C47.1
- net +1.875V: now also C45.1
- net +2.1875V: now also C46.1
- net 3.3V: now also C50.1, C51.1, C52.2
- net Clk_PostFanout_2: now also U18.6 (Y4); no longer U18.16 (Y1)
- net Clk_PostFanout_3: now also U18.8 (Y6); no longer U18.13 (Y2)
- net Clk_PostFanout_4: now also U18.11 (Y5); no longer U18.15 (Y3)
- net Clk_PostFanout_5: now also U18.13 (Y2); no longer U18.6 (Y4)
- net Clk_PostFanout_6: now also U18.15 (Y3); no longer U18.11 (Y5)
- net Clk_PostFanout_7: now also U18.16 (Y1); no longer U18.8 (Y6)
- net GND: now also C43.2, C44.2, C45.2, C46.2, C47.2, C48.2, C49.2, C50.2, C51.2, C52.1
- net PostRecieveClk renamed ComparatorClock
Other:
- moved on the sheet: C29, C30, C31, C32, C33, C34, C35, C36, C37, C38, C39, C40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

Commit message: board rev. 1.1
Parts:
- C29, C30, C31, C32, C33, C34, C35, C36, C37, C38, C39, C40, C41, C42, C43, C44, C45, C46, C47, C48, C49, C50, C51, C52: LCSC (none) -> C1591
- R29, R30, R31, R32, R33, R34, R35, R36: value 100(0.1%) -> 100; LCSC (none) -> C122970
- U10, U11, U12, U13, U14, U15, U16: LCSC (none) -> C207991
- U18: LCSC (none) -> C560966
