File: MixedSignal/PIO.kicad_sch (KiCad schematic)
At the start: 41 parts, among them J4 Input Audio Jack, J5 SDS-50J, U10LDO1 TPS7A4901DGNR, U20 AP2112K-3.3TRG1, U4 WE-TVS-82400102 TVS Diode Arr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, U8 REF5025AD, U9 OPA1612AxD, U9LDO1 TPS7A3001DGN

Commit message: passing DRC
Parts:
- removed R5(0.1%)1, R5(0.1%)2: 110k, Resistor_SMD:R_0603_1608Metric, symbol Device:R_US
- removed R6(0.1%)1, R6(0.1%)2: 12k, Resistor_SMD:R_0603_1608Metric, symbol Device:R_US
- added R10, R9: 110k (0.1%), Resistor_SMD:R_0603_1608Metric, symbol Device:R_US
- added R7, R8: 12k (0.1%), Resistor_SMD:R_0603_1608Metric, symbol Device:R_US
- R5(1%)1: value 150, 3W+ Load, move far from sensitive components, close to port -> 150, 3W+ Load, move far from sensitive components, close to port, 1%
- R5(1%)2: renamed from R5(1%)3; value 150, 3W+ Load, move far from sensitive components, close to port -> 150, 3W+ Load, move far from sensitive components, close to port, 1%
- U1: renamed from U9; footprint Package_SO:SOIC-8-1EP_3.9x4.9mm_P1.27mm_EP2.29x3mm -> Package_SO:SOIC-8_3.9x4.9mm_P1.27mm
- U10LDO1: footprint DGN8_1P89X1P57 -> TPS7A49:DGN8_1P89X1P57
- U9LDO1: footprint ADCComparator:DGN8_1P89X1P57 -> TPS7A49:DGN8_1P89X1P57
- renumbered C11 to C1, C12 to C10, C16 to C11, C9 to C12, C5 to C13, C3 to C14, C8 to C15, C4 to C16, C2 to C17, C7 to C18, C6 to C19, C18 to C2, C42 to C20, C1 to C3, C17 to C4, C13 to C5, C19 to C6, C14 to C7, C10 to C8, C15 to C9, J4 to J3, J5 to J4, R6 to R1, R5 to R2, R1 to R3, R2 to R4, R3 to R5, R4 to R6, U4 to U2, U8 to U3, U20 to U4
Connections:
- net +12V: now also R9.2
- net -12V: now also R10.2
- net GND: now also R7.1, R8.1
- net at U10LDO1.2 (FB): now also R7.2, R9.1
- net at U9LDO1.2 (FB): now also R10.1, R8.2

Commit message: board rev. 1.1
Parts:
- added C53: 0.1µF Ceramic, Capacitor_SMD:C_0603_1608Metric, symbol Device:C
- added D1, D2: STATUS, Diode_SMD:D_0603_1608Metric, symbol Device:D
- added FB2: Ferrite Bead, Diode_SMD:D_0603_1608Metric, symbol Device:FerriteBead
- added J5: B2B-XH-ALFSN, B2BHeader:CONN_B2B-XH-ALFSN_JST, symbol B2BHeader:B2B-XH-ALFSN
- C1: value 100µF Electrolytic (25V) -> 100µF Electrolytic; LCSC (none) -> C47344183
- C10, C8: value 100µF Electrolytic (25V) close to port -> 100µF Electrolytic; LCSC (none) -> C47344183
- C11: LCSC (none) -> C1588
- C12: LCSC (none) -> C15849
- C13, C14, C18, C19, C2, C6: value 10µF X7R Ceramic -> 10µF Ceramic; LCSC (none) -> C84416
- C15, C20: LCSC (none) -> C84416
- C16, C17: value 50nF -> 0.1µF Ceramic; LCSC (none) -> C1591
- C3, C4, C5, C7, C9: LCSC (none) -> C1591
- FB1: value FerriteBead -> Ferrite Bead; footprint Inductor_SMD:L_1206_3216Metric -> Diode_SMD:D_0603_1608Metric; LCSC (none) -> C14709
- J3: LCSC (none) -> C4991872
- J4: value SDS-50J -> DIN5 Connector; LCSC (none) -> C6216157
- R1, R2: value 1k(0.1%) -> 10k; LCSC (none) -> C25804
- R10, R9: value 110k (0.1%) -> 100k; LCSC (none) -> C25803
- R3, R4: value 100 -> 13k; LCSC (none) -> C22797
- R37: renamed from R5(1%)1; value 150, 3W+ Load, move far from sensitive components, close to port, 1% -> 150; LCSC (none) -> C479476
- R38: renamed from R5(1%)2; value 150, 3W+ Load, move far from sensitive components, close to port, 1% -> 150; LCSC (none) -> C479476
- R5, R6: LCSC (none) -> C25804
- R7, R8: value 12k (0.1%) -> 12k; LCSC (none) -> C22790
- U1: LCSC (none) -> C94590
- U10LDO1: LCSC (none) -> C16430
- U2: LCSC (none) -> C7519
- U3: LCSC (none) -> C523999
- U4: LCSC (none) -> C51118
- U9LDO1: value TPS7A3001DGN -> TPS7A3001DGNR; LCSC (none) -> C33835
Connections:
- net +1.25V: now also U1.5 (+); no longer U1.6 (-), U1.7
- net +12V: now also C53.2
- net +15V: now also R2.2
- net +2.5V: no longer R1.2
- net -15V: now also R1.2
- net 5V: now also FB2.1
- net GND: now also C53.1, D1.1 (K), D2.2 (A), J5.2; no longer R2.1
- new net: U1.6 (-), U1.7
- new net: D1.2 (A), R2.1
- new net: D2.1 (K), R1.1
- new net 5VOut: FB2.2, J5.1
Other:
- moved on the sheet: U1B
