File: MixedSignal/afe.kicad_sch (KiCad schematic)
At the start: 31 parts, among them U1 ADG734, U10 ADG734, U2 ADG734, U3 ADG734, U5 OPA1612AxD

Commit message: passing DRC
Parts:
- U7: renamed from U5; footprint Package_SO:SOIC-8-1EP_3.9x4.9mm_P1.27mm_EP2.29x3mm -> Package_SO:SOIC-8_3.9x4.9mm_P1.27mm
- renumbered C20 to C21, C21 to C22, C24 to C23, C25 to C24, C22 to C25, C23 to C28, R7 to R11, R9 to R12, R10 to R13, R11 to R14, R12 to R15, R13 to R16, R14 to R17, R15 to R18, R8 to R19, R16 to R20, R17 to R21, R18 to R22, R19 to R23, R20 to R24, R21 to R25, R22 to R26, R23 to R27, R24 to R28, U1 to U5, U2 to U6, U3 to U8, U10 to U9
Connections:
- net 3.3V: now also C27.1; no longer C27.2
- net DAC_CTRL_1: now also U8.20; no longer U8.1
- net DAC_CTRL_2: now also U8.11; no longer U8.10
- net DAC_CTRL_3: now also U8.10; no longer U8.11
- net DAC_CTRL_4: now also U8.1; no longer U8.20
- net DAC_CTRL_5: now also U9.20; no longer U9.1
- net DAC_CTRL_6: now also U9.11; no longer U9.10
- net DAC_CTRL_7: now also U9.10; no longer U9.11
- net DAC_CTRL_8: now also U9.1; no longer U9.20
- net FB_2.1: now also U8.18; no longer U8.3
- net FB_2.2: now also U8.13; no longer U8.8
- net FB_2.3: now also U8.8; no longer U8.13
- net FB_2.4: now also U8.3; no longer U8.18
- net FB_2.5: now also U9.18; no longer U9.3
- net FB_2.6: now also U9.13; no longer U9.8
- net FB_2.7: now also U9.8; no longer U9.13
- net FB_2.8: now also U9.3; no longer U9.18
- net GND: now also C27.2; no longer C27.1
Other:
- moved on the sheet: C27

Commit message: board rev. 1.1
Parts:
- removed R20: 16.9k, Resistor_SMD:R_0603_1608Metric, symbol Device:R_US
- removed R28: 13k, Resistor_SMD:R_0603_1608Metric, symbol Device:R_US
- added C54, C55, C56, C57, C58, C61, C62: 0.1µF Ceramic, Capacitor_SMD:C_0603_1608Metric, symbol Device:C
- added C59, C60: 10µF Ceramic, Capacitor_SMD:C_0805_2012Metric, symbol Device:C
- C21, C22, C23, C24, C26, C27: LCSC (none) -> C1591
- C25, C28: value 47pF -> 100pF; LCSC (none) -> C14858
- R11: value 2.8k -> 1.5k; LCSC (none) -> C22843
- R12, R13, R14, R15, R16, R17, R18: value 16.9k -> 14k; LCSC (none) -> C855621
- R19: value 1.62k -> 1.5k; LCSC (none) -> C22843
- R21, R22, R23, R24, R25, R26, R27: value 13k -> 7.32k; LCSC (none) -> C862286
- U5, U6, U8, U9: LCSC (none) -> C579105
- U7: LCSC (none) -> C94590
Connections:
- net FB_1.8 is gone; now on net FB_1.5: U6.18
- net FB_2.8 is gone; now on net GND: U9.3
- net +1.25V: now also C54.2
- net +2.5V: now also C55.2, C56.2, C57.2, C58.2, C59.2, C60.2, C61.2, C62.2; no longer U6.2, U9.4
- net FB_1.5: no longer U6.3
- net GND: now also U6.1, U6.2, U6.3, U9.1, U9.4, C54.1, C55.1, C56.1, C57.1, C58.1, C59.1, C60.1, C61.1, C62.1
- net DAC_CTRL_5 renamed DAC_CTRL_5B
- net DAC_CTRL_5B: no longer U6.1
- net DAC_CTRL_6 renamed DAC_CTRL_6A
- net DAC_CTRL_6A: no longer U9.11
- net DAC_CTRL_7 renamed DAC_CTRL_7A
- net DAC_CTRL_7A: no longer U9.10
- net DAC_CTRL_8 renamed DAC_CTRL_5A
- net DAC_CTRL_5A: no longer U9.1
- new net DAC_CTRL_6B: U9.11
- new net DAC_CTRL_7B: U9.10
